File: MRCS-555-Tone-Generator.sch (EAGLE design)
At the start: 16 parts, among them CON1 5V input, CON2 5 V input, CON3 output 3.5mm, CON4 Output 0.100, IC1 NE555

Commit message: Updates after first article tested good
clean up of some nomenclature
Parts:
- C1: value 0.01 uF 103 -> .01uF
- C4: value 0.01 103 -> 0.01uF
- C6: value 0.01 uF 103 -> 0.01uF
Changed lines of the file:
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@@
 <setting verticaltext="up"/>
 </settings>
-<grid distance="0.1" unitdist="inch" unit="inch" style="dots" multiple="1" display="yes" altdistance="50" altunitdist="mil" altunit="mil"/>
+<grid distance="100" unitdist="mil" unit="mil" style="dots" multiple="1" display="yes" altdistance="50" altunitdist="mil" altunit="mil"/>
 <layers>
 <layer number="1" name="Top" color="4" fill="1" visible="no" active="no"/>
@@
 <part name="R1" library="SPCoast" deviceset="R*" device="PTH04" value="100K"/>
 <part name="C2" library="SPCoast" deviceset="CAP-POL*" device="PTH-3.5MM" value="100 uF"/>
-<part name="C4" library="SPCoast" deviceset="CAP*" device="PTH2" value="0.01 103"/>
+<part name="C4" library="SPCoast" deviceset="CAP*" device="PTH2" value="0.01uF"/>
 <part name="R3" library="MRCS" deviceset="TRIM_US-" device="RS3" value="100K"/>
 <part name="CON1" library="SPCoast" deviceset="CONNECTOR-DC-POWER" device="-RA" value="5V input"/>
 <part name="CON4" library="SPCoast" deviceset="CONNECTOR-M02" device="1X02-LOCK" value="Output 0.100"/>
-<part name="C1" library="SPCoast" deviceset="CAP*" device="PTH2" value="0.01 uF 103"/>
+<part name="C1" library="SPCoast" deviceset="CAP*" device="PTH2" value=".01uF"/>
 <part name="P+3" library="SPCoast" deviceset="+5V" device=""/>
 <part name="GND4" library="SPCoast" deviceset="GND" device=""/>
 <part name="GND5" library="SPCoast" deviceset="GND" device=""/>
-<part name="C6" library="SPCoast" deviceset="CAP*" device="PTH2" value="0.01 uF 103"/>
+<part name="C6" library="SPCoast" deviceset="CAP*" device="PTH2" value="0.01uF "/>
 <part name="C5" library="SPCoast" deviceset="CAP-POL*" device="PTH-3.5MM" value="100 uF"/>
 <part name="P+2" library="SPCoast" deviceset="+5V" device=""/>
@@
 <instance part="C1" gate="C1" x="116.84" y="101.6" smashed="yes" rot="R90">
 <attribute name="NAME" x="131.064" y="106.045" size="1.778" layer="95" rot="R180"/>
-<attribute name="VALUE" x="141.224" y="103.251" size="1.778" layer="96" rot="R180"/>
+<attribute name="VALUE" x="131.064" y="103.251" size="1.778" layer="96" rot="R180"/>
 </instance>
 <instance part="P+3" gate="1" x="208.28" y="121.92"/>

Commit message: Minor updates after building 1st articles
Changed C3 from electrolytic to 0.1 for Tant or Monolithic
Minor clean up of labels on board
Parts:
- C1: value .01uF -> 0.01uF
- C3: device SPCoast:CAP-POLPTH-3.5MM -> SPCoast:CAPPTH2
Connections:
- net GND: now also C3.2; no longer C3.-
- net N$6: now also C3.1; no longer C3.+
Other:
- note added: "Seth Neumann"
Changed lines of the file:
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@@
 <part name="CON1" library="SPCoast" deviceset="CONNECTOR-DC-POWER" device="-RA" value="5V input"/>
 <part name="CON4" library="SPCoast" deviceset="CONNECTOR-M02" device="1X02-LOCK" value="Output 0.100"/>
-<part name="C1" library="SPCoast" deviceset="CAP*" device="PTH2" value=".01uF"/>
+<part name="C1" library="SPCoast" deviceset="CAP*" device="PTH2" value="0.01uF"/>
 <part name="P+3" library="SPCoast" deviceset="+5V" device=""/>
 <part name="GND4" library="SPCoast" deviceset="GND" device=""/>
@@
 <part name="P+2" library="SPCoast" deviceset="+5V" device=""/>
 <part name="GND2" library="SPCoast" deviceset="GND" device=""/>
-<part name="C3" library="SPCoast" deviceset="CAP-POL*" device="PTH-3.5MM" value="10 uF"/>
+<part name="C3" library="SPCoast" deviceset="CAP*" device="PTH2" value="10 uF"/>
 <part name="GND3" library="SPCoast" deviceset="GND" device=""/>
 </parts>
@@
 <plain>
 <text x="269.24" y="109.22" size="1.778" layer="91" rot="R90">output to speaker</text>
+<text x="175.26" y="25.4" size="2.54" layer="91">Seth Neumann</text>
 </plain>
 <instances>
@@
 <pinref part="GND2" gate="1" pin="GND"/>
 <wire x1="154.94" y1="116.84" x2="154.94" y2="99.06" width="0.6096" layer="91"/>
-<pinref part="C3" gate="C1" pin="-"/>
+<pinref part="C3" gate="C1" pin="2"/>
 <wire x1="162.56" y1="116.84" x2="154.94" y2="116.84" width="0.6096" layer="91"/>
 <junction x="154.94" y="116.84"/>
@@
 <wire x1="210.82" y1="129.54" x2="162.56" y2="129.54" width="0.3048" layer="91"/>
 <junction x="154.94" y="129.54"/>
-<pinref part="C3" gate="C1" pin="+"/>
+<pinref part="C3" gate="C1" pin="1"/>
 <wire x1="162.56" y1="129.54" x2="154.94" y2="129.54" width="0.3048" layer="91"/>
 <wire x1="162.56" y1="124.46" x2="162.56" y2="129.54" width="0.3048" layer="91"/>
